File: schm & pcb/8-bitCPU.kicad_sch (KiCad schematic)
At the start: 0 parts

Commit message: update from mac
Other:
- sheet ALU ports: added A_0, A_1, A_2, A_3, A_4, A_5, A_6, A_7, BUS_0, BUS_1, BUS_2, BUS_3, BUS_4, BUS_5, BUS_6, BUS_7, B_0, B_1, B_2, B_3, B_4, B_5, B_6, B_7, CF, CLK, CLR, SUB, ZF, ~{EO}, ~{FI}; removed none
- sheet Instruction Register ports: added BUS_0, BUS_1, BUS_2, BUS_3, BUS_4, BUS_5, BUS_6, BUS_7, CLEAR, CLK, I_4, I_5, I_6, I_7, ~{II}, ~{IO}; removed none
- sheet Memory Address Register ports: added BUS_0, BUS_1, BUS_2, BUS_3, CLK, CLR, MA0, MA1, MA2, MA3, PROG, ~{MI}; removed none
- sheet Output Register ports: added BUS_0, BUS_1, BUS_2, BUS_3, BUS_4, BUS_5, BUS_6, BUS_7, CLK, OI, ~{CLR}; removed none
- sheet Random Access Memory ports: added BUS_0, BUS_1, BUS_2, BUS_3, BUS_4, BUS_5, BUS_6, BUS_7, CLK, MA0, MA1, MA2, MA3, PROG, RI, ~{RO}; removed none
