File: schm & pcb/clock.kicad_sch (KiCad schematic)
At the start: 28 parts

Commit message: update from mac
Parts:
- gave numbers to parts that had none: 24
Changed lines of the file:
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@@
   (symbol (lib_id "Timer:LM555xN") (at 56.515 66.675 0) (unit 1)
     (in_bom yes) (on_board yes)
-    (property "Reference" "U?" (id 0) (at 47.625 57.785 0)
+    (property "Reference" "U1" (id 0) (at 47.625 57.785 0)
       (effects (font (size 1.27 1.27)) (justify left))
     )
@@
   (symbol (lib_id "Device:C") (at 213.995 78.105 0) (unit 1)
     (in_bom yes) (on_board yes)
-    (property "Reference" "C?" (id 0) (at 216.535 76.835 0)
+    (property "Reference" "C5" (id 0) (at 216.535 76.835 0)
       (effects (font (size 1.27 1.27)) (justify left))
     )
@@
   (symbol (lib_id "74xx:74LS04") (at 188.595 123.825 0) (unit 3)
     (in_bom yes) (on_board yes) (fields_autoplaced)
-    (property "Reference" "U?" (id 0) (at 188.595 114.935 0))
+    (property "Reference" "U2" (id 0) (at 188.595 114.935 0))
     (property "Value" "74LS04" (id 1) (at 188.595 117.475 0))
     (property "Footprint" "" (id 2) (at 188.595 123.825 0)
@@
   (symbol (lib_id "Timer:LM555xN") (at 146.685 66.675 0) (unit 1)
     (in_bom yes) (on_board yes)
-    (property "Reference" "U?" (id 0) (at 137.795 57.785 0)
+    (property "Reference" "U5" (id 0) (at 137.795 57.785 0)
       (effects (font (size 1.27 1.27)) (justify left))
     )
@@
   (symbol (lib_id "Device:R") (at 205.105 51.435 0) (unit 1)
     (in_bom yes) (on_board yes)
-    (property "Reference" "R?" (id 0) (at 206.375 50.165 0)
+    (property "Reference" "R6" (id 0) (at 206.375 50.165 0)
       (effects (font (size 1.27 1.27)) (justify left))
     )
@@
   (symbol (lib_id "Device:C") (at 128.905 78.105 0) (unit 1)
     (in_bom yes) (on_board yes)
-    (property "Reference" "C?" (id 0) (at 131.445 76.835 0)
+    (property "Reference" "C3" (id 0) (at 131.445 76.835 0)
       (effects (font (size 1.27 1.27)) (justify left))
     )
@@
   (symbol (lib_id "Device:R") (at 160.655 53.975 0) (unit 1)
     (in_bom yes) (on_board yes)
-    (property "Reference" "R?" (id 0) (at 161.925 52.705 0)
+    (property "Reference" "R4" (id 0) (at 161.925 52.705 0)
       (effects (font (size 1.27 1.27)) (justify left))
     )
@@
   (symbol (lib_id "power:GND") (at 146.685 86.995 0) (unit 1)
     (in_bom yes) (on_board yes)
-    (property "Reference" "#PWR0108" (id 0) (at 146.685 93.345 0)
+    (property "Reference" "#PWR0109" (id 0) (at 146.685 93.345 0)
       (effects (font (size 1.27 1.27)) hide)
     )
@@
   (symbol (lib_id "74xx:74LS04") (at 85.725 136.525 0) (unit 2)
     (in_bom yes) (on_board yes) (fields_autoplaced)
-    (property "Reference" "U?" (id 0) (at 85.725 127.635 0))
+    (property "Reference" "U2" (id 0) (at 85.725 127.635 0))
     (property "Value" "74LS04" (id 1) (at 85.725 130.175 0))
     (property "Footprint" "" (id 2) (at 85.725 136.525 0)
@@
   (symbol (lib_id "74xx:74LS08") (at 160.655 132.715 0) (unit 3)
     (in_bom yes) (on_board yes) (fields_autoplaced)
-    (property "Reference" "U?" (id 0) (at 160.655 123.825 0))
+    (property "Reference" "U3" (id 0) (at 160.655 123.825 0))
     (property "Value" "74LS08" (id 1) (at 160.655 126.365 0))
     (property "Footprint" "" (id 2) (at 160.655 132.715 0)
@@
   (symbol (lib_id "74xx:74LS04") (at 130.175 149.225 0) (unit 1)
     (in_bom yes) (on_board yes) (fields_autoplaced)
-    (property "Reference" "U?" (id 0) (at 130.175 140.335 0))
+    (property "Reference" "U2" (id 0) (at 130.175 140.335 0))
     (property "Value" "74LS04" (id 1) (at 130.175 142.875 0))
     (property "Footprint" "" (id 2) (at 130.175 149.225 0)
@@
   (symbol (lib_id "Device:C") (at 250.825 32.385 0) (unit 1)
     (in_bom yes) (on_board yes)
-    (property "Reference" "C?" (id 0) (at 253.365 31.115 0)
+    (property "Reference" "C6" (id 0) (at 253.365 31.115 0)
       (effects (font (size 1.27 1.27)) (justify left))
     )
@@
   (symbol (lib_id "74xx:74LS08") (at 107.315 139.065 0) (unit 2)
     (in_bom yes) (on_board yes) (fields_autoplaced)
-    (property "Reference" "U?" (id 0) (at 107.315 130.175 0))
+    (property "Reference" "U3" (id 0) (at 107.315 130.175 0))
     (property "Value" "74LS08" (id 1) (at 107.315 132.715 0))
     (property "Footprint" "" (id 2) (at 107.315 139.065 0)
@@
   (symbol (lib_id "Device:LED") (at 182.245 139.065 90) (unit 1)
     (in_bom yes) (on_board yes)
-    (property "Reference" "D?" (id 0) (at 184.785 137.795 90)
+    (property "Reference" "D1" (id 0) (at 184.785 137.795 90)
       (effects (font (size 1.27 1.27)) (justify right))
     )
@@
   (symbol (lib_id "Device:C_Polarized") (at 38.735 83.185 0) (unit 1)
     (in_bom yes) (on_board yes)
-    (property "Reference" "C?" (id 0) (at 41.275 81.915 0)
+    (property "Reference" "C2" (id 0) (at 41.275 81.915 0)
       (effects (font (size 1.27 1.27)) (justify left))
     )
@@
   (symbol (lib_id "Device:C") (at 260.985 32.385 0) (unit 1)
     (in_bom yes) (on_board yes)
-    (property "Reference" "C?" (id 0) (at 263.525 31.115 0)
+    (property "Reference" "C7" (id 0) (at 263.525 31.115 0)
       (effects (font (size 1.27 1.27)) (justify left))
     )
@@
   (symbol (lib_id "Device:R_Potentiometer") (at 88.265 66.675 180) (unit 1)
     (in_bom yes) (on_board yes)
-    (property "Reference" "RV?" (id 0) (at 89.535 65.405 0)
+    (property "Reference" "RV1" (id 0) (at 89.535 65.405 0)
       (effects (font (size 1.27 1.27)) (justify right))
     )
@@
   (symbol (lib_id "Device:R") (at 128.905 55.245 0) (unit 1)
     (in_bom yes) (on_board yes)
-    (property "Reference" "R?" (id 0) (at 125.095 53.975 0)
+    (property "Reference" "R3" (id 0) (at 125.095 53.975 0)
       (effects (font (size 1.27 1.27)) (justify left))
     )
@@
   (symbol (lib_id "Device:C") (at 32.385 83.185 0) (unit 1)
     (in_bom yes) (on_board yes)
-    (property "Reference" "C?" (id 0) (at 27.305 80.645 0)
+    (property "Reference" "C1" (id 0) (at 27.305 80.645 0)
       (effects (font (size 1.27 1.27)) (justify left))
     )
@@
   (symbol (lib_id "Timer:LM555xN") (at 229.235 66.675 0) (unit 1)
     (in_bom yes) (on_board yes)
-    (property "Reference" "U?" (id 0) (at 220.345 57.785 0)
+    (property "Reference" "U6" (id 0) (at 220.345 57.785 0)
       (effects (font (size 1.27 1.27)) (justify left))
     )
@@
   (symbol (lib_id "74xx:74LS32") (at 131.445 130.175 0) (unit 1)
     (in_bom yes) (on_board yes) (fields_autoplaced)
-    (property "Reference" "U?" (id 0) (at 131.445 121.285 0))
+    (property "Reference" "U4" (id 0) (at 131.445 121.285 0))
     (property "Value" "74LS32" (id 1) (at 131.445 123.825 0))
     (property "Footprint" "" (id 2) (at 131.445 130.175 0)
@@
   (symbol (lib_id "Switch:SW_Push") (at 121.285 61.595 0) (unit 1)
     (in_bom yes) (on_board yes)
-    (property "Reference" "SW?" (id 0) (at 117.475 59.055 0))
+    (property "Reference" "SW1" (id 0) (at 117.475 59.055 0))
     (property "Value" "SW_Push" (id 1) (at 121.285 64.135 0))
     (property "Footprint" "" (id 2) (at 121.285 56.515 0)
@@
   (symbol (lib_id "Switch:SW_SPDT") (at 197.485 64.135 0) (unit 1)
     (in_bom yes) (on_board yes) (fields_autoplaced)
-    (property "Reference" "SW?" (id 0) (at 197.485 56.515 0))
+    (property "Reference" "SW2" (id 0) (at 197.485 56.515 0))
     (property "Value" "SW_SPDT" (id 1) (at 197.485 59.055 0))
     (property "Footprint" "" (id 2) (at 197.485 64.135 0)
@@
   (symbol (lib_id "Device:R") (at 79.375 66.675 90) (unit 1)
     (in_bom yes) (on_board yes)
-    (property "Reference" "R?" (id 0) (at 79.375 64.135 90))
+    (property "Reference" "R2" (id 0) (at 79.375 64.135 90))
     (property "Value" "1K" (id 1) (at 79.375 69.215 90))
     (property "Footprint" "" (id 2) (at 79.375 68.453 90)
@@
   (symbol (lib_id "power:+5V") (at 56.515 47.625 0) (unit 1)
     (in_bom yes) (on_board yes)
-    (property "Reference" "#PWR0109" (id 0) (at 56.515 51.435 0)
+    (property "Reference" "#PWR0108" (id 0) (at 56.515 51.435 0)
       (effects (font (size 1.27 1.27)) hide)
     )
@@
   (symbol (lib_id "74xx:74LS08") (at 108.585 121.285 0) (unit 1)
     (in_bom yes) (on_board yes) (fields_autoplaced)
-    (property "Reference" "U?" (id 0) (at 108.585 112.395 0))
+    (property "Reference" "U3" (id 0) (at 108.585 112.395 0))
     (property "Value" "74LS08" (id 1) (at 108.585 114.935 0))
     (property "Footprint" "" (id 2) (at 108.585 121.285 0)
@@
   (symbol (lib_id "Device:R") (at 211.455 51.435 0) (unit 1)
     (in_bom yes) (on_board yes)
-    (property "Reference" "R?" (id 0) (at 212.725 50.165 0)
+    (property "Reference" "R7" (id 0) (at 212.725 50.165 0)
       (effects (font (size 1.27 1.27)) (justify left))
     )
@@
   (symbol (lib_id "Device:R") (at 182.245 147.955 0) (unit 1)
     (in_bom yes) (on_board yes)
-    (property "Reference" "R?" (id 0) (at 183.515 146.685 0)
+    (property "Reference" "R5" (id 0) (at 183.515 146.685 0)
       (effects (font (size 1.27 1.27)) (justify left))
     )
@@
   (symbol (lib_id "Device:R") (at 71.755 53.975 0) (unit 1)
     (in_bom yes) (on_board yes)
-    (property "Reference" "R?" (id 0) (at 73.025 52.705 0)
+    (property "Reference" "R1" (id 0) (at 73.025 52.705 0)
       (effects (font (size 1.27 1.27)) (justify left))
     )
@@
   (symbol (lib_id "Device:C") (at 160.655 78.105 0) (unit 1)
     (in_bom yes) (on_board yes)
-    (property "Reference" "C?" (id 0) (at 163.195 76.835 0)
-      (effects (font (size 1.27 1.27)) (justify left))
-    )
+    (property "Reference" "C4" (id 0) (at 163.195 76.835 0)
+      (effects (font (size 1.27 1.27)) (justify left))
+    )
