File: schm & pcb/controlLogic.kicad_sch (KiCad schematic)
At the start: 0 parts

Commit message: update from mac
Parts:
- added C15, C16: C, symbol Device:C
- added D54, D55, D56, D57, D58, D59, D60, D61, D62, D63, D64, D65, D66, D67, D68, D69, D70, D71, D72, D73, D74, D75, D76, D77, D78, D79: LED, symbol Device:LED
- added R64, R77, R79, R81: R, symbol Device:R
- added R65, R66, R67, R68, R69, R70, R71, R72, R73, R74, R75, R76, R78, R80, R82, R83, R84, R85, R86, R87, R88, R89, R90: 220, symbol Device:R
- added SW8: SW_Push, symbol Switch:SW_Push
- added U27, U47: 74LS00, symbol 74xx:74LS00
- added U29, U30, U52, U53: 74LS04, symbol 74xx:74LS04
- added U48: 74LS161, symbol 74xx:74LS161
- added U49: 74LS138, symbol 74xx:74LS138
- added U50, U51: AT28C16, Package_DIP:DIP-24_W15.24mm_LongPads, symbol Memory_EEPROM:AT28C16
Connections:
- new net: D70.1 (K), R82.1
- new net: D70.2 (A), U51.17 (I/O7), U53.1
- new net: D75.2 (A), U30.5, U50.13 (I/O3)
- new net: D54.2 (A), R66.1
- new net: D56.2 (A), R68.1
- new net: D72.1 (K), R83.1
- new net: D60.1 (K), R71.1
- new net: D60.2 (A), U51.11 (I/O2), U52.5
- new net: D66.1 (K), R74.2
- new net: R64.1, SW8.1, U27.10, U27.9
- new net: D78.1 (K), R89.1
- new net: D68.1 (K), R80.1
- new net: D76.1 (K), R87.1
- new net: D76.2 (A), U50.14 (I/O4), U52.3
- new net: D73.2 (A), U29.11, U50.10 (I/O1)
- new net: D74.2 (A), U29.9, U50.11 (I/O2)
- new net: D78.2 (A), U50.16 (I/O6), U52.1
- new net: U50.6 (A2), U51.6 (A2)
- new net: U50.7 (A1), U51.7 (A1)
- new net: U50.8 (A0), U51.8 (A0)
- new net: D72.2 (A), U29.13, U50.9 (I/O0)
- new net: D75.1 (K), R86.1
- new net: D55.2 (A), R67.1
- new net: D57.2 (A), R69.1
- new net: D58.1 (K), R65.1
- new net: D58.2 (A), U30.11, U51.9 (I/O0)
- new net: D62.1 (K), R76.1
- new net: D61.1 (K), R72.1
- new net: D73.1 (K), R84.1
- new net: U27.12, U27.13, U27.4, U27.8
- new net: U27.5, U49.10 (O5)
- new net: D65.1 (K), R73.2
- new net: D74.1 (K), R85.1
- new net: D59.1 (K), R70.1
- new net: D59.2 (A), U30.9, U51.10 (I/O1)
- new net: U47.3, U48.1 (~{MR})
- new net: D67.1 (K), R75.2
- new net: D63.1 (K), R78.1
- new net: U27.6, U47.1, U47.2
- new net: D77.1 (K), R88.1
- new net: D63.2 (A), U51.15 (I/O5), U53.3
- new net: D79.1 (K), R90.1
- new net +5V: R66.2, R67.2, R68.2, R69.2, U51.24 (VCC)
- new net CE: D61.2 (A), U51.13 (I/O3)
- new net GND: R65.2, R70.2, R71.2, R72.2, R76.2, R78.2, R80.2, R82.2, R83.2, R84.2, R85.2, R86.2, R87.2, R88.2, R89.2, R90.2
- new net HLT: D79.2 (A), U50.17 (I/O7)
- new net OI: D62.2 (A), U51.14 (I/O4)
- new net Ri: D77.2 (A), U50.15 (I/O5)
- new net SU: D68.2 (A), U51.16 (I/O6)
- new net ~{AI}: U29.10
- new net ~{AO}: U29.12
- new net ~{BI}: U53.4
- new net ~{CO}: U52.6
- new net ~{EO}: U53.2
- new net ~{FI}: U30.10
- new net ~{II}: U29.8
- new net ~{IO}: U30.6
- new net ~{J}: U30.8
- new net ~{MI}: U52.2
- new net ~{RO}: U52.4
