File: schm & pcb/instructionRegister.kicad_sch (KiCad schematic)
At the start: 19 parts

Commit message: update from mac
Parts:
- gave numbers to parts that had none: 19
Changed lines of the file:
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@@
   (symbol (lib_id "Device:LED") (at 90.17 146.05 90) (unit 1)
     (in_bom yes) (on_board yes)
-    (property "Reference" "D?" (id 0) (at 91.44 144.78 90)
+    (property "Reference" "D18" (id 0) (at 91.44 144.78 90)
       (effects (font (size 1.27 1.27)) (justify right))
     )
@@
   (symbol (lib_id "Device:R") (at 118.11 156.21 0) (unit 1)
     (in_bom yes) (on_board yes)
-    (property "Reference" "R?" (id 0) (at 119.38 154.305 0)
+    (property "Reference" "R28" (id 0) (at 119.38 154.305 0)
       (effects (font (size 1.27 1.27)) (justify left))
     )
@@
   (symbol (lib_id "Device:R") (at 90.17 156.21 0) (unit 1)
     (in_bom yes) (on_board yes)
-    (property "Reference" "R?" (id 0) (at 91.44 154.305 0)
+    (property "Reference" "R24" (id 0) (at 91.44 154.305 0)
       (effects (font (size 1.27 1.27)) (justify left))
     )
@@
   (symbol (lib_id "Device:LED") (at 97.155 146.05 90) (unit 1)
     (in_bom yes) (on_board yes)
-    (property "Reference" "D?" (id 0) (at 98.425 144.78 90)
+    (property "Reference" "D19" (id 0) (at 98.425 144.78 90)
       (effects (font (size 1.27 1.27)) (justify right))
     )
@@
   (symbol (lib_id "Device:LED") (at 132.08 146.05 90) (unit 1)
     (in_bom yes) (on_board yes)
-    (property "Reference" "D?" (id 0) (at 133.35 144.78 90)
+    (property "Reference" "D24" (id 0) (at 133.35 144.78 90)
       (effects (font (size 1.27 1.27)) (justify right))
     )
@@
   (symbol (lib_id "Device:R") (at 125.095 156.21 0) (unit 1)
     (in_bom yes) (on_board yes)
-    (property "Reference" "R?" (id 0) (at 126.365 154.305 0)
+    (property "Reference" "R29" (id 0) (at 126.365 154.305 0)
       (effects (font (size 1.27 1.27)) (justify left))
     )
@@
   (symbol (lib_id "Device:LED") (at 118.11 146.05 90) (unit 1)
     (in_bom yes) (on_board yes)
-    (property "Reference" "D?" (id 0) (at 119.38 144.78 90)
+    (property "Reference" "D22" (id 0) (at 119.38 144.78 90)
       (effects (font (size 1.27 1.27)) (justify right))
     )
@@
   (symbol (lib_id "Device:LED") (at 139.065 146.05 90) (unit 1)
     (in_bom yes) (on_board yes)
-    (property "Reference" "D?" (id 0) (at 140.335 144.78 90)
+    (property "Reference" "D25" (id 0) (at 140.335 144.78 90)
       (effects (font (size 1.27 1.27)) (justify right))
     )
@@
   (symbol (lib_id "Device:LED") (at 104.14 146.05 90) (unit 1)
     (in_bom yes) (on_board yes)
-    (property "Reference" "D?" (id 0) (at 105.41 144.78 90)
+    (property "Reference" "D20" (id 0) (at 105.41 144.78 90)
       (effects (font (size 1.27 1.27)) (justify right))
     )
@@
   (symbol (lib_id "Device:LED") (at 125.095 146.05 90) (unit 1)
     (in_bom yes) (on_board yes)
-    (property "Reference" "D?" (id 0) (at 126.365 144.78 90)
+    (property "Reference" "D23" (id 0) (at 126.365 144.78 90)
       (effects (font (size 1.27 1.27)) (justify right))
     )
@@
   (symbol (lib_id "74xx:74LS245") (at 78.74 83.82 90) (unit 1)
     (in_bom yes) (on_board yes)
-    (property "Reference" "U?" (id 0) (at 93.345 74.93 90))
+    (property "Reference" "U13" (id 0) (at 93.345 74.93 90))
     (property "Value" "74LS245" (id 1) (at 96.52 92.71 90))
     (property "Footprint" "" (id 2) (at 78.74 83.82 0)
@@
   (symbol (lib_id "Device:R") (at 132.08 156.21 0) (unit 1)
     (in_bom yes) (on_board yes)
-    (property "Reference" "R?" (id 0) (at 133.35 154.305 0)
+    (property "Reference" "R30" (id 0) (at 133.35 154.305 0)
       (effects (font (size 1.27 1.27)) (justify left))
     )
@@
   (symbol (lib_id "74xx:74LS173") (at 143.51 83.82 270) (unit 1)
     (in_bom yes) (on_board yes)
-    (property "Reference" "U?" (id 0) (at 160.655 74.93 90))
+    (property "Reference" "U14" (id 0) (at 160.655 74.93 90))
     (property "Value" "74LS173" (id 1) (at 164.465 92.71 90))
     (property "Footprint" "" (id 2) (at 143.51 83.82 0)
@@
   (symbol (lib_id "74xx:74LS173") (at 209.55 84.455 270) (unit 1)
     (in_bom yes) (on_board yes)
-    (property "Reference" "U?" (id 0) (at 226.695 75.565 90))
+    (property "Reference" "U15" (id 0) (at 226.695 75.565 90))
     (property "Value" "74LS173" (id 1) (at 229.87 93.345 90))
     (property "Footprint" "" (id 2) (at 209.55 84.455 0)
@@
   (symbol (lib_id "Device:R") (at 104.14 156.21 0) (unit 1)
     (in_bom yes) (on_board yes)
-    (property "Reference" "R?" (id 0) (at 105.41 154.305 0)
+    (property "Reference" "R26" (id 0) (at 105.41 154.305 0)
       (effects (font (size 1.27 1.27)) (justify left))
     )
@@
   (symbol (lib_id "Device:LED") (at 111.125 146.05 90) (unit 1)
     (in_bom yes) (on_board yes)
-    (property "Reference" "D?" (id 0) (at 112.395 144.78 90)
+    (property "Reference" "D21" (id 0) (at 112.395 144.78 90)
       (effects (font (size 1.27 1.27)) (justify right))
     )
@@
   (symbol (lib_id "Device:R") (at 139.065 156.21 0) (unit 1)
     (in_bom yes) (on_board yes)
-    (property "Reference" "R?" (id 0) (at 140.335 154.305 0)
+    (property "Reference" "R31" (id 0) (at 140.335 154.305 0)
       (effects (font (size 1.27 1.27)) (justify left))
     )
@@
   (symbol (lib_id "Device:R") (at 97.155 156.21 0) (unit 1)
     (in_bom yes) (on_board yes)
-    (property "Reference" "R?" (id 0) (at 98.425 154.305 0)
+    (property "Reference" "R25" (id 0) (at 98.425 154.305 0)
       (effects (font (size 1.27 1.27)) (justify left))
     )
@@
   (symbol (lib_id "Device:R") (at 111.125 156.21 0) (unit 1)
     (in_bom yes) (on_board yes)
-    (property "Reference" "R?" (id 0) (at 112.395 154.305 0)
-      (effects (font (size 1.27 1.27)) (justify left))
-    )
+    (property "Reference" "R27" (id 0) (at 112.395 154.305 0)
+      (effects (font (size 1.27 1.27)) (justify left))
+    )
