File: schm & pcb/mar.kicad_sch (KiCad schematic)
At the start: 17 parts

Commit message: update from mac
Parts:
- gave numbers to parts that had none: 17
Changed lines of the file:
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@@
   (symbol (lib_id "74xx:74LS157") (at 140.335 73.66 90) (unit 1)
     (in_bom yes) (on_board yes)
-    (property "Reference" "U?" (id 0) (at 160.02 64.135 90))
+    (property "Reference" "U24" (id 0) (at 160.02 64.135 90))
     (property "Value" "74LS157" (id 1) (at 163.83 82.55 90))
     (property "Footprint" "" (id 2) (at 140.335 73.66 0)
@@
   (symbol (lib_id "Device:LED") (at 82.55 50.165 90) (unit 1)
     (in_bom yes) (on_board yes)
-    (property "Reference" "D?" (id 0) (at 83.82 48.26 90)
+    (property "Reference" "D37" (id 0) (at 83.82 48.26 90)
       (effects (font (size 1.27 1.27)) (justify right))
     )
@@
   (symbol (lib_id "Switch:SW_SPDT") (at 65.405 93.345 0) (unit 1)
     (in_bom yes) (on_board yes) (fields_autoplaced)
-    (property "Reference" "SW?" (id 0) (at 65.405 85.725 0))
+    (property "Reference" "SW3" (id 0) (at 65.405 85.725 0))
     (property "Value" "SW_SPDT" (id 1) (at 65.405 88.265 0))
     (property "Footprint" "" (id 2) (at 65.405 93.345 0)
@@
   (symbol (lib_id "power:GND") (at 54.61 97.79 0) (unit 1)
     (in_bom yes) (on_board yes)
-    (property "Reference" "#PWR0166" (id 0) (at 54.61 104.14 0)
+    (property "Reference" "#PWR0167" (id 0) (at 54.61 104.14 0)
       (effects (font (size 1.27 1.27)) hide)
     )
@@
   (symbol (lib_id "Device:LED") (at 86.995 102.87 270) (unit 1)
     (in_bom yes) (on_board yes)
-    (property "Reference" "D?" (id 0) (at 85.725 104.775 90)
+    (property "Reference" "D38" (id 0) (at 85.725 104.775 90)
       (effects (font (size 1.27 1.27)) (justify right))
     )
@@
   (symbol (lib_id "power:GND") (at 92.71 68.58 0) (unit 1)
     (in_bom yes) (on_board yes)
-    (property "Reference" "#PWR0138" (id 0) (at 92.71 74.93 0)
+    (property "Reference" "#PWR0162" (id 0) (at 92.71 74.93 0)
       (effects (font (size 1.27 1.27)) hide)
     )
@@
   (symbol (lib_id "Device:LED") (at 103.505 50.165 90) (unit 1)
     (in_bom yes) (on_board yes)
-    (property "Reference" "D?" (id 0) (at 104.775 48.26 90)
+    (property "Reference" "D41" (id 0) (at 104.775 48.26 90)
       (effects (font (size 1.27 1.27)) (justify right))
     )
@@
   (symbol (lib_id "Device:R") (at 96.52 60.96 0) (unit 1)
     (in_bom yes) (on_board yes)
-    (property "Reference" "R?" (id 0) (at 97.79 59.69 0)
+    (property "Reference" "R46" (id 0) (at 97.79 59.69 0)
       (effects (font (size 1.27 1.27)) (justify left))
     )
@@
   (symbol (lib_id "Connector_Generic:Conn_01x04") (at 165.1 133.35 0) (unit 1)
     (in_bom yes) (on_board yes) (fields_autoplaced)
-    (property "Reference" "J?" (id 0) (at 167.64 133.3499 0)
+    (property "Reference" "J1" (id 0) (at 167.64 133.3499 0)
       (effects (font (size 1.27 1.27)) (justify left))
     )
@@
   (symbol (lib_id "power:GND") (at 158.115 87.63 0) (unit 1)
     (in_bom yes) (on_board yes)
-    (property "Reference" "#PWR0137" (id 0) (at 158.115 93.98 0)
+    (property "Reference" "#PWR0159" (id 0) (at 158.115 93.98 0)
       (effects (font (size 1.27 1.27)) hide)
     )
@@
   (symbol (lib_id "Device:R") (at 80.01 112.395 180) (unit 1)
     (in_bom yes) (on_board yes)
-    (property "Reference" "R?" (id 0) (at 78.74 113.665 0)
+    (property "Reference" "R42" (id 0) (at 78.74 113.665 0)
       (effects (font (size 1.27 1.27)) (justify left))
     )
@@
   (symbol (lib_id "power:+5V") (at 241.935 69.85 0) (unit 1)
     (in_bom yes) (on_board yes) (fields_autoplaced)
-    (property "Reference" "#PWR0167" (id 0) (at 241.935 73.66 0)
+    (property "Reference" "#PWR0165" (id 0) (at 241.935 73.66 0)
       (effects (font (size 1.27 1.27)) hide)
     )
@@
   (symbol (lib_id "power:GND") (at 190.5 73.025 0) (unit 1)
     (in_bom yes) (on_board yes)
-    (property "Reference" "#PWR0170" (id 0) (at 190.5 79.375 0)
+    (property "Reference" "#PWR0160" (id 0) (at 190.5 79.375 0)
       (effects (font (size 1.27 1.27)) hide)
     )
@@
   (symbol (lib_id "power:GND") (at 124.46 121.285 0) (unit 1)
     (in_bom yes) (on_board yes)
-    (property "Reference" "#PWR0171" (id 0) (at 124.46 127.635 0)
+    (property "Reference" "#PWR0158" (id 0) (at 124.46 127.635 0)
       (effects (font (size 1.27 1.27)) hide)
     )
@@
   (symbol (lib_id "Device:LED") (at 80.01 102.87 270) (unit 1)
     (in_bom yes) (on_board yes)
-    (property "Reference" "D?" (id 0) (at 78.74 104.775 90)
+    (property "Reference" "D36" (id 0) (at 78.74 104.775 90)
       (effects (font (size 1.27 1.27)) (justify right))
     )
@@
   (symbol (lib_id "power:GND") (at 168.91 75.565 0) (unit 1)
     (in_bom yes) (on_board yes)
-    (property "Reference" "#PWR0169" (id 0) (at 168.91 81.915 0)
+    (property "Reference" "#PWR0161" (id 0) (at 168.91 81.915 0)
       (effects (font (size 1.27 1.27)) hide)
     )
@@
   (symbol (lib_id "Device:R") (at 86.995 112.395 180) (unit 1)
     (in_bom yes) (on_board yes)
-    (property "Reference" "R?" (id 0) (at 85.725 113.665 0)
+    (property "Reference" "R44" (id 0) (at 85.725 113.665 0)
       (effects (font (size 1.27 1.27)) (justify left))
     )
@@
   (symbol (lib_id "power:+5V") (at 114.935 72.39 0) (unit 1)
     (in_bom yes) (on_board yes) (fields_autoplaced)
-    (property "Reference" "#PWR0173" (id 0) (at 114.935 76.2 0)
+    (property "Reference" "#PWR0163" (id 0) (at 114.935 76.2 0)
       (effects (font (size 1.27 1.27)) hide)
     )
@@
   (symbol (lib_id "Device:R") (at 82.55 60.96 0) (unit 1)
     (in_bom yes) (on_board yes)
-    (property "Reference" "R?" (id 0) (at 83.82 59.69 0)
+    (property "Reference" "R43" (id 0) (at 83.82 59.69 0)
       (effects (font (size 1.27 1.27)) (justify left))
     )
@@
   (symbol (lib_id "power:+5V") (at 93.98 118.11 0) (unit 1)
     (in_bom yes) (on_board yes) (fields_autoplaced)
-    (property "Reference" "#PWR0165" (id 0) (at 93.98 121.92 0)
+    (property "Reference" "#PWR0166" (id 0) (at 93.98 121.92 0)
       (effects (font (size 1.27 1.27)) hide)
     )
@@
   (symbol (lib_id "Switch:SW_DIP_x04") (at 130.81 133.35 270) (unit 1)
     (in_bom yes) (on_board yes)
-    (property "Reference" "SW?" (id 0) (at 139.065 128.27 90)
+    (property "Reference" "SW4" (id 0) (at 139.065 128.27 90)
       (effects (font (size 1.27 1.27)) (justify left))
     )
@@
   (symbol (lib_id "power:GND") (at 134.62 145.415 0) (unit 1)
     (in_bom yes) (on_board yes)
-    (property "Reference" "#PWR0172" (id 0) (at 134.62 151.765 0)
+    (property "Reference" "#PWR0157" (id 0) (at 134.62 151.765 0)
       (effects (font (size 1.27 1.27)) hide)
     )
@@
   (symbol (lib_id "Device:R") (at 103.505 60.96 0) (unit 1)
     (in_bom yes) (on_board yes)
-    (property "Reference" "R?" (id 0) (at 104.775 59.69 0)
+    (property "Reference" "R47" (id 0) (at 104.775 59.69 0)
       (effects (font (size 1.27 1.27)) (justify left))
     )
@@
   (symbol (lib_id "Device:LED") (at 96.52 50.165 90) (unit 1)
     (in_bom yes) (on_board yes)
-    (property "Reference" "D?" (id 0) (at 97.79 48.26 90)
+    (property "Reference" "D40" (id 0) (at 97.79 48.26 90)
       (effects (font (size 1.27 1.27)) (justify right))
     )
@@
   (symbol (lib_id "power:GND") (at 212.725 48.895 0) (unit 1)
     (in_bom yes) (on_board yes)
-    (property "Reference" "#PWR0168" (id 0) (at 212.725 55.245 0)
+    (property "Reference" "#PWR0164" (id 0) (at 212.725 55.245 0)
       (effects (font (size 1.27 1.27)) hide)
     )
@@
   (symbol (lib_id "Device:R") (at 89.535 60.96 0) (unit 1)
     (in_bom yes) (on_board yes)
-    (property "Reference" "R?" (id 0) (at 90.805 59.69 0)
+    (property "Reference" "R45" (id 0) (at 90.805 59.69 0)
       (effects (font (size 1.27 1.27)) (justify left))
     )
@@
   (symbol (lib_id "74xx:74LS173") (at 215.9 71.755 270) (unit 1)
     (in_bom yes) (on_board yes)
-    (property "Reference" "U?" (id 0) (at 233.68 62.23 90))
+    (property "Reference" "U25" (id 0) (at 233.68 62.23 90))
     (property "Value" "74LS173" (id 1) (at 236.22 81.28 90))
     (property "Footprint" "" (id 2) (at 215.9 71.755 0)
@@
   (symbol (lib_id "Device:LED") (at 89.535 50.165 90) (unit 1)
     (in_bom yes) (on_board yes)
-    (property "Reference" "D?" (id 0) (at 90.805 48.26 90)
-      (effects (font (size 1.27 1.27)) (justify right))
-    )
+    (property "Reference" "D39" (id 0) (at 90.805 48.26 90)
+      (effects (font (size 1.27 1.27)) (justify right))
+    )
