File: schm & pcb/pc.kicad_sch (KiCad schematic)
At the start: 10 parts

Commit message: update from mac
Parts:
- gave numbers to parts that had none: 10
Changed lines of the file:
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@@
   (symbol (lib_id "Device:R") (at 120.015 142.875 0) (unit 1)
     (in_bom yes) (on_board yes)
-    (property "Reference" "R?" (id 0) (at 121.285 141.605 0)
+    (property "Reference" "R60" (id 0) (at 121.285 141.605 0)
       (effects (font (size 1.27 1.27)) (justify left))
     )
@@
   (symbol (lib_id "power:GND") (at 109.22 150.495 0) (unit 1)
     (in_bom yes) (on_board yes)
-    (property "Reference" "#PWR0142" (id 0) (at 109.22 156.845 0)
+    (property "Reference" "#PWR0192" (id 0) (at 109.22 156.845 0)
       (effects (font (size 1.27 1.27)) hide)
     )
@@
   (symbol (lib_id "74xx:74LS245") (at 73.66 92.075 90) (unit 1)
     (in_bom yes) (on_board yes)
-    (property "Reference" "U?" (id 0) (at 86.995 83.185 90))
+    (property "Reference" "U35" (id 0) (at 86.995 83.185 90))
     (property "Value" "74LS245" (id 1) (at 91.44 100.965 90))
     (property "Footprint" "" (id 2) (at 73.66 92.075 0)
@@
   (symbol (lib_id "power:GND") (at 83.82 106.045 0) (unit 1)
     (in_bom yes) (on_board yes)
-    (property "Reference" "#PWR0141" (id 0) (at 83.82 112.395 0)
+    (property "Reference" "#PWR0191" (id 0) (at 83.82 112.395 0)
       (effects (font (size 1.27 1.27)) hide)
     )
@@
   (symbol (lib_id "power:+5V") (at 163.195 92.075 0) (unit 1)
     (in_bom yes) (on_board yes)
-    (property "Reference" "#PWR0144" (id 0) (at 163.195 95.885 0)
+    (property "Reference" "#PWR0194" (id 0) (at 163.195 95.885 0)
       (effects (font (size 1.27 1.27)) hide)
     )
@@
   (symbol (lib_id "Device:LED") (at 106.045 132.08 90) (unit 1)
     (in_bom yes) (on_board yes)
-    (property "Reference" "D?" (id 0) (at 107.315 130.175 90)
+    (property "Reference" "D51" (id 0) (at 107.315 130.175 90)
       (effects (font (size 1.27 1.27)) (justify right))
     )
@@
   (symbol (lib_id "74xx:74LS161") (at 140.97 92.71 270) (unit 1)
     (in_bom yes) (on_board yes)
-    (property "Reference" "U?" (id 0) (at 155.575 83.82 90))
+    (property "Reference" "U36" (id 0) (at 155.575 83.82 90))
     (property "Value" "74LS161" (id 1) (at 158.75 102.235 90))
     (property "Footprint" "" (id 2) (at 140.97 92.71 0)
@@
   (symbol (lib_id "Device:LED") (at 120.015 132.08 90) (unit 1)
     (in_bom yes) (on_board yes)
-    (property "Reference" "D?" (id 0) (at 121.285 130.175 90)
+    (property "Reference" "D53" (id 0) (at 121.285 130.175 90)
       (effects (font (size 1.27 1.27)) (justify right))
     )
@@
   (symbol (lib_id "Device:LED") (at 99.06 132.08 90) (unit 1)
     (in_bom yes) (on_board yes)
-    (property "Reference" "D?" (id 0) (at 100.33 130.175 90)
+    (property "Reference" "D50" (id 0) (at 100.33 130.175 90)
       (effects (font (size 1.27 1.27)) (justify right))
     )
@@
   (symbol (lib_id "Device:R") (at 113.03 142.875 0) (unit 1)
     (in_bom yes) (on_board yes)
-    (property "Reference" "R?" (id 0) (at 114.3 141.605 0)
+    (property "Reference" "R59" (id 0) (at 114.3 141.605 0)
       (effects (font (size 1.27 1.27)) (justify left))
     )
@@
   (symbol (lib_id "power:+5V") (at 52.07 90.805 0) (unit 1)
     (in_bom yes) (on_board yes)
-    (property "Reference" "#PWR0140" (id 0) (at 52.07 94.615 0)
+    (property "Reference" "#PWR0190" (id 0) (at 52.07 94.615 0)
       (effects (font (size 1.27 1.27)) hide)
     )
@@
   (symbol (lib_id "power:GND") (at 118.11 93.98 0) (unit 1)
     (in_bom yes) (on_board yes)
-    (property "Reference" "#PWR0143" (id 0) (at 118.11 100.33 0)
+    (property "Reference" "#PWR0193" (id 0) (at 118.11 100.33 0)
       (effects (font (size 1.27 1.27)) hide)
     )
@@
   (symbol (lib_id "power:GND") (at 96.52 93.345 0) (unit 1)
     (in_bom yes) (on_board yes)
-    (property "Reference" "#PWR0139" (id 0) (at 96.52 99.695 0)
+    (property "Reference" "#PWR0189" (id 0) (at 96.52 99.695 0)
       (effects (font (size 1.27 1.27)) hide)
     )
@@
   (symbol (lib_id "Device:R") (at 99.06 142.875 0) (unit 1)
     (in_bom yes) (on_board yes)
-    (property "Reference" "R?" (id 0) (at 100.33 141.605 0)
+    (property "Reference" "R57" (id 0) (at 100.33 141.605 0)
       (effects (font (size 1.27 1.27)) (justify left))
     )
@@
   (symbol (lib_id "Device:R") (at 106.045 142.875 0) (unit 1)
     (in_bom yes) (on_board yes)
-    (property "Reference" "R?" (id 0) (at 107.315 141.605 0)
+    (property "Reference" "R58" (id 0) (at 107.315 141.605 0)
       (effects (font (size 1.27 1.27)) (justify left))
     )
@@
   (symbol (lib_id "Device:LED") (at 113.03 132.08 90) (unit 1)
     (in_bom yes) (on_board yes)
-    (property "Reference" "D?" (id 0) (at 114.3 130.175 90)
-      (effects (font (size 1.27 1.27)) (justify right))
-    )
+    (property "Reference" "D52" (id 0) (at 114.3 130.175 90)
+      (effects (font (size 1.27 1.27)) (justify right))
+    )
