File: schm & pcb/ram.kicad_sch (KiCad schematic)
At the start: 0 parts

Commit message: update from mac
Parts:
- added C10, C9: 0.1uF, symbol Device:C
- added C8: 0.01uF, symbol Device:C
- added D42, D43, D44, D45, D46, D47, D48, D49: LED, symbol Device:LED
- added J2: Conn_01x08, symbol Connector_Generic:Conn_01x08
- added R48, R49, R51, R52, R53, R54, R55, R56: 220, symbol Device:R
- added R50: 1k, symbol Device:R
- added SW5: SW_Push, symbol Switch:SW_Push
- added SW6: SW_DIP_x08, symbol Switch:SW_DIP_x08
- added U2, U29, U30: 74LS04, symbol 74xx:74LS04
- added U26, U33, U34: 74LS157, symbol 74xx:74LS157
- added U27: 74LS00, symbol 74xx:74LS00
- added U28, U31: 74189, Package_DIP:DIP-12_W7.62mm_LongPads, symbol 74xx:74189
- added U32: 74LS245, symbol 74xx:74LS245
Connections:
- new net: C8.2, R50.1, U27.2
- new net: U30.1, U31.7 (~{O1})
- new net: D48.2 (A), U30.2, U32.8 (A6)
- new net: U26.10 (I1c), U27.3
- new net: J2.1 (Pin_1), SW6.1, U34.14 (I0d)
- new net: J2.7 (Pin_7), SW6.10, U33.5 (I0b)
- new net: J2.4 (Pin_4), SW6.13, U34.2 (I0a)
- new net: J2.3 (Pin_3), SW6.14, U34.5 (I0b)
- new net: J2.2 (Pin_2), SW6.2, U34.11 (I0c)
- new net: J2.5 (Pin_5), SW6.5, U33.14 (I0d)
- new net: J2.6 (Pin_6), SW6.6, U33.11 (I0c)
- new net: J2.8 (Pin_8), SW6.9, U33.2 (I0a)
- new net: D45.1 (K), R52.1
- new net: SW5.2, U26.11 (I0c)
- new net: D47.2 (A), U2.12, U32.7 (A5)
- new net: U2.13, U31.9 (~{O2})
- new net: D45.2 (A), U2.8, U32.5 (A3)
- new net: U28.9 (~{O2}), U29.5
- new net: D44.2 (A), U29.6, U32.4 (A2)
- new net: D48.1 (K), R55.1
- new net: D47.1 (K), R54.1
- new net: D44.1 (K), R51.1
- new net: U28.7 (~{O1}), U29.3
- new net: D43.2 (A), U29.4, U32.3 (A1)
- new net: U30.3, U31.5 (~{O0})
- new net: D49.2 (A), U30.4, U32.9 (A7)
- new net: D43.1 (K), R49.1
- new net: U2.9, U28.11 (~{O3})
- new net: D46.1 (K), R53.1
- new net: D49.1 (K), R56.1
- new net: D46.2 (A), U2.10, U32.6 (A4)
- new net: D42.1 (K), R48.1
- new net: U2.11, U31.11 (~{O3})
- new net: U26.9 (Zc), U28.3 (~{WE}), U31.3 (~{WE})
- new net: U28.5 (~{O0}), U29.1
- new net: U31.10 (D2), U34.9 (Zc)
- new net: U31.12 (D3), U34.12 (Zd)
- new net: U31.4 (D0), U34.4 (Za)
- new net: U31.6 (D1), U34.7 (Zb)
- new net: D42.2 (A), U29.2, U32.2 (A0)
- new net +5V: C10.1, C9.1, U26.16 (VCC), U28.16 (VCC), U31.16 (VCC), U32.1 (A->B), U32.20 (VCC), U33.16 (VCC), U34.16 (VCC)
- new net BUS_0: U32.11 (B7), U34.13 (I1d)
- new net BUS_1: U32.12 (B6), U34.10 (I1c)
- new net BUS_2: U32.13 (B5), U34.6 (I1b)
- new net BUS_3: U32.14 (B4), U34.3 (I1a)
- new net BUS_4: U32.15 (B3), U33.13 (I1d)
- new net BUS_5: U32.16 (B2), U33.10 (I1c)
- new net BUS_6: U32.17 (B1), U33.6 (I1b)
- new net BUS_7: U32.18 (B0), U33.3 (I1a)
- new net CLK: C8.1
- new net D5: U28.12 (D3), U33.12 (Zd)
- new net D6: U28.10 (D2), U33.9 (Zc)
- new net D7: U28.6 (D1), U33.7 (Zb)
- new net D8: U28.4 (D0), U33.4 (Za)
- new net GND: C10.2, C9.2, R48.2, R49.2, R50.2, R51.2, R52.2, R53.2, R54.2, R55.2, R56.2, SW5.1, SW6.11, SW6.12, SW6.15, SW6.16, SW6.3, SW6.4, SW6.7, SW6.8, U26.15 (E), U26.8 (GND), U28.2 (~{CS}), U28.8 (GND), U31.2 (~{CS}), U31.8 (GND), U32.10 (GND), U33.15 (E), U33.8 (GND), U34.15 (E), U34.8 (GND)
- new net MA0: U28.1 (A0), U31.1 (A0)
- new net MA1: U28.15 (A1), U31.15 (A1)
- new net MA2: U28.14 (A2), U31.14 (A2)
- new net MA3: U28.13 (A3), U31.13 (A3)
- new net PROG: U26.1 (S), U33.1 (S), U34.1 (S)
- new net RI: U27.1
- new net ~{RO}: U32.19 (CE)
- no-connect marks 0 -> 9
