File: schm & pcb/registerA.kicad_sch (KiCad schematic)
At the start: 19 parts

Commit message: update from mac
Parts:
- D2, D3, D4, D5, D6, D7, D8, D9: renamed from D?; value (none) -> LED
- R10, R11, R12, R13, R14, R15, R8, R9: renamed from R?; value (none) -> 220
- U7: renamed from U?; value (none) -> 74LS245
- U8, U9: renamed from U?; value (none) -> 74LS173
