File: schm & pcb/registerB.kicad_sch (KiCad schematic)
At the start: 19 parts

Commit message: update from mac
Parts:
- gave numbers to parts that had none: 19
Changed lines of the file:
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@@
     (stroke (width 0) (type default) (color 0 0 0 0))
   )
-  (hierarchical_label "B_4" (shape input) (at 147.955 131.445 0)
-    (effects (font (size 1.27 1.27)) (justify left))
-  )
-  (hierarchical_label "BUS_1" (shape input) (at 41.275 31.115 180)
-    (effects (font (size 1.27 1.27)) (justify right))
-  )
-  (hierarchical_label "B_0" (shape input) (at 147.955 123.825 0)
+  (hierarchical_label "B_4" (shape output) (at 147.955 131.445 0)
+    (effects (font (size 1.27 1.27)) (justify left))
+  )
+  (hierarchical_label "BUS_1" (shape bidirectional) (at 41.275 31.115 180)
+    (effects (font (size 1.27 1.27)) (justify right))
+  )
+  (hierarchical_label "B_0" (shape output) (at 147.955 123.825 0)
     (effects (font (size 1.27 1.27)) (justify left))
   )
@@
     (effects (font (size 1.27 1.27)) (justify right))
   )
-  (hierarchical_label "BUS_4" (shape input) (at 41.275 38.735 180)
-    (effects (font (size 1.27 1.27)) (justify right))
-  )
-  (hierarchical_label "BUS_6" (shape input) (at 41.275 43.815 180)
+  (hierarchical_label "BUS_4" (shape bidirectional) (at 41.275 38.735 180)
+    (effects (font (size 1.27 1.27)) (justify right))
+  )
+  (hierarchical_label "BUS_6" (shape bidirectional) (at 41.275 43.815 180)
     (effects (font (size 1.27 1.27)) (justify right))
   )
@@
     (effects (font (size 1.27 1.27)) (justify right))
   )
-  (hierarchical_label "BUS_3" (shape input) (at 41.275 36.195 180)
-    (effects (font (size 1.27 1.27)) (justify right))
-  )
-  (hierarchical_label "B_5" (shape input) (at 147.955 133.35 0)
-    (effects (font (size 1.27 1.27)) (justify left))
-  )
-  (hierarchical_label "BUS_2" (shape input) (at 41.275 33.655 180)
-    (effects (font (size 1.27 1.27)) (justify right))
-  )
-  (hierarchical_label "BUS_5" (shape input) (at 41.275 41.275 180)
-    (effects (font (size 1.27 1.27)) (justify right))
-  )
-  (hierarchical_label "B_3" (shape input) (at 147.955 129.54 0)
-    (effects (font (size 1.27 1.27)) (justify left))
-  )
-  (hierarchical_label "B_7" (shape input) (at 147.955 137.16 0)
-    (effects (font (size 1.27 1.27)) (justify left))
-  )
-  (hierarchical_label "BUS_7" (shape input) (at 41.275 46.355 180)
-    (effects (font (size 1.27 1.27)) (justify right))
-  )
-  (hierarchical_label "B_6" (shape input) (at 147.955 135.255 0)
+  (hierarchical_label "BUS_3" (shape bidirectional) (at 41.275 36.195 180)
+    (effects (font (size 1.27 1.27)) (justify right))
+  )
+  (hierarchical_label "B_5" (shape output) (at 147.955 133.35 0)
+    (effects (font (size 1.27 1.27)) (justify left))
+  )
+  (hierarchical_label "BUS_2" (shape bidirectional) (at 41.275 33.655 180)
+    (effects (font (size 1.27 1.27)) (justify right))
+  )
+  (hierarchical_label "BUS_5" (shape bidirectional) (at 41.275 41.275 180)
+    (effects (font (size 1.27 1.27)) (justify right))
+  )
+  (hierarchical_label "B_3" (shape output) (at 147.955 129.54 0)
+    (effects (font (size 1.27 1.27)) (justify left))
+  )
+  (hierarchical_label "B_7" (shape output) (at 147.955 137.16 0)
+    (effects (font (size 1.27 1.27)) (justify left))
+  )
+  (hierarchical_label "BUS_7" (shape bidirectional) (at 41.275 46.355 180)
+    (effects (font (size 1.27 1.27)) (justify right))
+  )
+  (hierarchical_label "B_6" (shape output) (at 147.955 135.255 0)
     (effects (font (size 1.27 1.27)) (justify left))
   )
@@
     (effects (font (size 1.27 1.27)) (justify left))
   )
-  (hierarchical_label "B_2" (shape input) (at 147.955 127.635 0)
-    (effects (font (size 1.27 1.27)) (justify left))
-  )
-  (hierarchical_label "B_1" (shape input) (at 147.955 125.73 0)
+  (hierarchical_label "B_2" (shape output) (at 147.955 127.635 0)
+    (effects (font (size 1.27 1.27)) (justify left))
+  )
+  (hierarchical_label "B_1" (shape output) (at 147.955 125.73 0)
     (effects (font (size 1.27 1.27)) (justify left))
   )
@@
     (effects (font (size 1.27 1.27)) (justify right))
   )
-  (hierarchical_label "BUS_0" (shape input) (at 41.275 28.575 180)
+  (hierarchical_label "BUS_0" (shape bidirectional) (at 41.275 28.575 180)
     (effects (font (size 1.27 1.27)) (justify right))
   )
@@
   (symbol (lib_id "74xx:74LS173") (at 208.28 87.63 270) (unit 1)
     (in_bom yes) (on_board yes)
-    (property "Reference" "U?" (id 0) (at 225.425 78.74 90))
+    (property "Reference" "U12" (id 0) (at 225.425 78.74 90))
     (property "Value" "74LS173" (id 1) (at 228.6 96.52 90))
     (property "Footprint" "" (id 2) (at 208.28 87.63 0)
@@
   (symbol (lib_id "Device:LED") (at 102.87 149.225 90) (unit 1)
     (in_bom yes) (on_board yes)
-    (property "Reference" "D?" (id 0) (at 104.14 147.955 90)
+    (property "Reference" "D12" (id 0) (at 104.14 147.955 90)
       (effects (font (size 1.27 1.27)) (justify right))
     )
@@
   (symbol (lib_id "Device:LED") (at 88.9 149.225 90) (unit 1)
     (in_bom yes) (on_board yes)
-    (property "Reference" "D?" (id 0) (at 90.17 147.955 90)
+    (property "Reference" "D10" (id 0) (at 90.17 147.955 90)
       (effects (font (size 1.27 1.27)) (justify right))
     )
@@
   (symbol (lib_id "Device:R") (at 123.825 159.385 0) (unit 1)
     (in_bom yes) (on_board yes)
-    (property "Reference" "R?" (id 0) (at 125.095 157.48 0)
+    (property "Reference" "R21" (id 0) (at 125.095 157.48 0)
       (effects (font (size 1.27 1.27)) (justify left))
     )
@@
   (symbol (lib_id "Device:LED") (at 130.81 149.225 90) (unit 1)
     (in_bom yes) (on_board yes)
-    (property "Reference" "D?" (id 0) (at 132.08 147.955 90)
+    (property "Reference" "D16" (id 0) (at 132.08 147.955 90)
       (effects (font (size 1.27 1.27)) (justify right))
     )
@@
   (symbol (lib_id "Device:R") (at 137.795 159.385 0) (unit 1)
     (in_bom yes) (on_board yes)
-    (property "Reference" "R?" (id 0) (at 139.065 157.48 0)
+    (property "Reference" "R23" (id 0) (at 139.065 157.48 0)
       (effects (font (size 1.27 1.27)) (justify left))
     )
@@
   (symbol (lib_id "74xx:74LS173") (at 142.24 86.995 270) (unit 1)
     (in_bom yes) (on_board yes)
-    (property "Reference" "U?" (id 0) (at 159.385 78.105 90))
+    (property "Reference" "U11" (id 0) (at 159.385 78.105 90))
     (property "Value" "74LS173" (id 1) (at 163.195 95.885 90))
     (property "Footprint" "" (id 2) (at 142.24 86.995 0)
@@
   (symbol (lib_id "Device:R") (at 130.81 159.385 0) (unit 1)
     (in_bom yes) (on_board yes)
-    (property "Reference" "R?" (id 0) (at 132.08 157.48 0)
+    (property "Reference" "R22" (id 0) (at 132.08 157.48 0)
       (effects (font (size 1.27 1.27)) (justify left))
     )
@@
   (symbol (lib_id "Device:R") (at 102.87 159.385 0) (unit 1)
     (in_bom yes) (on_board yes)
-    (property "Reference" "R?" (id 0) (at 104.14 157.48 0)
+    (property "Reference" "R18" (id 0) (at 104.14 157.48 0)
       (effects (font (size 1.27 1.27)) (justify left))
     )
@@
   (symbol (lib_id "74xx:74LS245") (at 77.47 86.995 90) (unit 1)
     (in_bom yes) (on_board yes)
-    (property "Reference" "U?" (id 0) (at 92.075 78.105 90))
+    (property "Reference" "U10" (id 0) (at 92.075 78.105 90))
     (property "Value" "74LS245" (id 1) (at 95.25 95.885 90))
     (property "Footprint" "" (id 2) (at 77.47 86.995 0)
@@
   (symbol (lib_id "Device:R") (at 116.84 159.385 0) (unit 1)
     (in_bom yes) (on_board yes)
-    (property "Reference" "R?" (id 0) (at 118.11 157.48 0)
+    (property "Reference" "R20" (id 0) (at 118.11 157.48 0)
       (effects (font (size 1.27 1.27)) (justify left))
     )
@@
   (symbol (lib_id "Device:LED") (at 109.855 149.225 90) (unit 1)
     (in_bom yes) (on_board yes)
-    (property "Reference" "D?" (id 0) (at 111.125 147.955 90)
+    (property "Reference" "D13" (id 0) (at 111.125 147.955 90)
       (effects (font (size 1.27 1.27)) (justify right))
     )
@@
   (symbol (lib_id "Device:R") (at 95.885 159.385 0) (unit 1)
     (in_bom yes) (on_board yes)
-    (property "Reference" "R?" (id 0) (at 97.155 157.48 0)
+    (property "Reference" "R17" (id 0) (at 97.155 157.48 0)
       (effects (font (size 1.27 1.27)) (justify left))
     )
@@
   (symbol (lib_id "Device:LED") (at 95.885 149.225 90) (unit 1)
     (in_bom yes) (on_board yes)
-    (property "Reference" "D?" (id 0) (at 97.155 147.955 90)
+    (property "Reference" "D11" (id 0) (at 97.155 147.955 90)
       (effects (font (size 1.27 1.27)) (justify right))
     )
@@
   (symbol (lib_id "Device:LED") (at 116.84 149.225 90) (unit 1)
     (in_bom yes) (on_board yes)
-    (property "Reference" "D?" (id 0) (at 118.11 147.955 90)
+    (property "Reference" "D14" (id 0) (at 118.11 147.955 90)
       (effects (font (size 1.27 1.27)) (justify right))
     )
@@
   (symbol (lib_id "Device:R") (at 88.9 159.385 0) (unit 1)
     (in_bom yes) (on_board yes)
-    (property "Reference" "R?" (id 0) (at 90.17 157.48 0)
+    (property "Reference" "R16" (id 0) (at 90.17 157.48 0)
       (effects (font (size 1.27 1.27)) (justify left))
     )
@@
   (symbol (lib_id "Device:R") (at 109.855 159.385 0) (unit 1)
     (in_bom yes) (on_board yes)
-    (property "Reference" "R?" (id 0) (at 111.125 157.48 0)
+    (property "Reference" "R19" (id 0) (at 111.125 157.48 0)
       (effects (font (size 1.27 1.27)) (justify left))
     )
@@
   (symbol (lib_id "Device:LED") (at 123.825 149.225 90) (unit 1)
     (in_bom yes) (on_board yes)
-    (property "Reference" "D?" (id 0) (at 125.095 147.955 90)
+    (property "Reference" "D15" (id 0) (at 125.095 147.955 90)
       (effects (font (size 1.27 1.27)) (justify right))
     )
@@
   (symbol (lib_id "Device:LED") (at 137.795 149.225 90) (unit 1)
     (in_bom yes) (on_board yes)
-    (property "Reference" "D?" (id 0) (at 139.065 147.955 90)
-      (effects (font (size 1.27 1.27)) (justify right))
-    )
+    (property "Reference" "D17" (id 0) (at 139.065 147.955 90)
+      (effects (font (size 1.27 1.27)) (justify right))
+    )
